Commit message: first commit

File: fishbot_description/urdf/fishbot/fishbot.urdf.xacro (robot description, xacro)
@@ -4,6 +4,6 @@
     <!-- 传感器组件 -->
     <xacro:include filename="$(find fishbot_description)/urdf/fishbot/sensor/imu.urdf.xacro" />
-    <xacro:include filename="$(find fishbot_description)/urdf/fishbot/sensor/laser.urdf.xacro" />
-    <xacro:include filename="$(find fishbot_description)/urdf/fishbot/sensor/camera.urdf.xacro" />
+    <!-- <xacro:include filename="$(find fishbot_description)/urdf/fishbot/sensor/laser.urdf.xacro" /> -->
+    <xacro:include filename="$(find ros2_livox_simulation)/urdf/mid360.xacro" />
      <!-- 执行器组件 -->
     <xacro:include filename="$(find fishbot_description)/urdf/fishbot/actuator/wheel.urdf.xacro" />
@@ -11,7 +11,9 @@
     <xacro:base_xacro length="0.12" radius="0.1" />
     <!-- 传感器 -->
-    <xacro:imu_xacro xyz="0 0 0.02" />
-    <xacro:laser_xacro xyz="0 0 0.10" />
-    <xacro:camera_xacro xyz="0.10 0 0.075" />
+    <xacro:imu_xacro xyz="0 0 0.05" />
+    <!-- <xacro:laser_xacro xyz="0 0 0.10" /> -->
+    <xacro:mid360 name="livox" parent="base_link" topic="mid360">
+        <origin xyz="0 0 0.08" rpy="0 0 0"/>
+    </xacro:mid360>
     <!-- 执行器主动轮+从动轮 -->
     <xacro:wheel_xacro wheel_name="left" xyz="0 0.10 -0.06" />

File: fishbot_description/urdf/fishbot/plugins/gazebo_sensor_plugin.xacro (robot description, xacro)
@@ -111,28 +111,3 @@
 </gazebo>
     </xacro:macro>
-<gazebo reference="camera_link">
-    <sensor type="depth" name="camera_sensor">
-        <plugin name="depth_camera" filename="libgazebo_ros_camera.so">
-            <frame_name>camera_optical_link</frame_name>
-        </plugin>
-        <always_on>true</always_on>
-        <update_rate>10</update_rate>
-        <camera name="camera">
-            <horizontal_fov>1.5009831567</horizontal_fov>
-            <image>
-                <width>800</width>
-                <height>600</height>
-                <format>R8G8B8</format>
-            </image>
-            <distortion>
-                <k1>0.0</k1>
-                <k2>0.0</k2>
-                <k3>0.0</k3>
-                <p1>0.0</p1>
-                <p2>0.0</p2>
-                <center>0.5 0.5</center>
-            </distortion>
-        </camera>
-    </sensor>
-</gazebo>
 </robot>
